File: kicad/pico_dow_clock/_restore_backup_2026-07-10T10-45-06-981/pico_dow_clock.kicad_sch (KiCad schematic)
At the start: 31 parts, among them Q2 AO3400A, SW1 SW_Push_Dual, U1 AMS1117-3.3

Commit message: LCD symbol update for new LCD
Parts:
- removed R19, R20, R21, R22, R23, R24: 15, symbol Device:R
- added R12, R13, R14, R15, R16, R17: 15, symbol Device:R
Connections:
- net +3.3V: now also LCD1.4 (DC), LCD2.4 (DC), LCD3.4 (DC), LCD4.4 (DC), LCD5.4 (DC), LCD6.4 (DC)
- net BL_POWER: now also R12.1, R13.1, R14.1, R15.1, R16.1, R17.1
- net LCD_CLK: now also LCD1.3 (RST), LCD2.3 (RST), LCD3.3 (RST), LCD4.3 (RST), LCD5.3 (RST), LCD6.3 (RST); no longer LCD1.6 (CLK), LCD2.6 (CLK), LCD3.6 (CLK), LCD4.6 (CLK), LCD5.6 (CLK), LCD6.6 (CLK)
- net LCD_DC: no longer LCD1.4 (DC), LCD2.4 (DC), LCD3.4 (DC), LCD4.4 (DC), LCD5.4 (DC), LCD6.4 (DC)
- net LCD_DIN: now also LCD1.1 (LEDA), LCD2.1 (LEDA), LCD3.1 (LEDA), LCD4.1 (LEDA), LCD5.1 (LEDA), LCD6.1 (LEDA); no longer LCD1.5 (DIN), LCD2.5 (DIN), LCD3.5 (DIN), LCD4.5 (DIN), LCD5.5 (DIN), LCD6.5 (DIN)
- net LCD1_CS_N renamed LCD_1_CS
- net LCD_1_CS: now also LCD1.6 (CLK); no longer LCD1.8 (~{CS})
- net LCD2_CS_N renamed LCD_2_CS
- net LCD_2_CS: now also LCD2.6 (CLK); no longer LCD2.8 (~{CS})
- net LCD3_CS_N renamed LCD_3_CS
- net LCD_3_CS: now also LCD3.6 (CLK); no longer LCD3.8 (~{CS})
- net LCD4_CS_N renamed LCD_4_CS
- net LCD_4_CS: now also LCD4.6 (CLK); no longer LCD4.8 (~{CS})
- net LCD5_CS_N renamed LCD_5_CS
- net LCD_5_CS: now also LCD5.6 (CLK); no longer LCD5.8 (~{CS})
- net LCD6_CS_N renamed LCD_6_CS
- net LCD_6_CS: now also LCD6.6 (CLK); no longer LCD6.8 (~{CS})
- net LCD7_CS_N renamed LCD_7_CS
- net LCD_7_CS: no longer LCD7.8 (~{CS})
- removed net LCD_RST_N: LCD1.3 (~{RST}), LCD2.3 (~{RST}), LCD3.3 (~{RST}), LCD4.3 (~{RST}), LCD5.3 (~{RST}), LCD6.3 (~{RST}), LCD7.3 (~{RST}), LEV1.18 (B1)
- net P_LCD_RST_N renamed P_LCD_RST
- new net: LCD5.5 (DIN), R16.2
- new net: LCD2.5 (DIN), R13.2
- new net: LCD3.5 (DIN), R14.2
- new net: LCD1.5 (DIN), R12.2
- new net: LCD4.5 (DIN), R15.2
- new net: LCD6.5 (DIN), R17.2
- new net LCD_CS_1: LCD7.8 (CS)
- new net LCD_RST: LCD1.8 (CS), LCD2.8 (CS), LCD3.8 (CS), LCD4.8 (CS), LCD5.8 (CS), LCD6.8 (CS), LCD7.3 (RST), LEV1.18 (B1)
Other:
- moved on the sheet: CPU1
