File: kicad/pico_dow_clock/pico_dow_clock.kicad_sch (KiCad schematic)
At the start: 31 parts, among them Q2 AO3400A, SW1 SW_Push_Dual, U1 AMS1117-3.3

Commit message: Add light sensor for ambient light
Parts:
- added Q1: TEPT4400, LED_THT:LED_D3.0mm_Clear, symbol Sensor_Optical:TEPT4400
- added R4: 50k, symbol Device:R
- D2: value LED_Dual_Bidirectional -> LED_Bidirectional
Connections:
- net +3.3V: now also Q1.1 (C)
- net GND: now also R4.1
- net AMB_LVL: now reaches CPU1.31 (GPIO26_ADC0)
- net AMB_LVL: now also Q1.2 (E), R4.2
- no-connect marks 30 -> 29
Other:
- note added: "Light Sensor"
- moved on the sheet: D2, LEV1, R1, R2
